File: design/micro.kicad_sch (KiCad schematic)
At the start: 15 parts, among them IC5 STM32L431CCT6TR, J2 Conn_ARM_SWD_TagConnect_TC203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, J3 Conn_01x02_Pin, J4 Conn_01x02_Pin, J5 Conn_01x02_Pin

Commit message: - Added display.kicad_sch; - Added mounting holes on schematic; - Removed TAG connect pads and used pin header; - Cut the PCB in order to make space for USB connector; - Changed mounting holes foorprint to non-plated ones; - Cut board near SHT4x sensor in order to reduce heat contribution from the rest of the board; - Re-routing; - Added revision number on silkscreen; - Shrunk components ID on silkscreen.
Parts:
- removed J2: Conn_ARM_SWD_TagConnect_TC2030-NL, Connector:Tag-Connect_TC2030-IDC-NL_2x03_P1.27mm_Vertical, symbol Connector:Conn_ARM_SWD_TagConnect_TC2030-NL
- added J7: Conn_01x06, Connector_PinHeader_2.54mm:PinHeader_1x06_P2.54mm_Vertical, symbol Connector_Generic:Conn_01x06
Connections:
- net MCU_NRST: now also J7.2 (Pin_2)
- net MCU_SWCLK: now also J7.3 (Pin_3)
- net MCU_SWDIO: now also J7.4 (Pin_4)
- net MCU_SWO: now also J7.5 (Pin_5)
- net VDD: now also J7.1 (Pin_1)
- net VSS: now also J7.6 (Pin_6)
Other:
- note added: "SWD Interface"
- note removed: "TODO: Mettere 6 header maschi"

Commit message: Updated 3D models of components; Addend new PCB renders; Updated README.md; Updated board to revision 2.0; Schematic and layout cleanup and minor changes.
Parts:
- J7: now left out of the parts list
Other:
- note removed: "ok"
Changed lines of the file:
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@@
 		(title "MCU schematic")
 		(date "2026-09-23")
-		(rev "1.1")
+		(rev "2.0")
 	)
 	(rectangle
@@
 		(exclude_from_sim no)
 		(at 39.624 162.56 0)
-		(effects
-			(font
-				(size 1.27 1.27)
-			)
-		)
-	)
-	(text "ok"
-		(exclude_from_sim no)
-		(at 236.982 133.858 0)
 		(effects
 			(font
@@
 		(body_style 1)
 		(exclude_from_sim no)
-		(in_bom yes)
+		(in_bom no)
 		(on_board yes)
 		(in_pos_files yes)
