File: design/usb.kicad_sch (KiCad schematic)
At the start: 15 parts, among them IC4 AZ1117CH-3.3TRG1, J1 UJ20-C-H-G-MSMT-4B-P16-TR

Commit message: - Added display.kicad_sch; - Added mounting holes on schematic; - Removed TAG connect pads and used pin header; - Cut the PCB in order to make space for USB connector; - Changed mounting holes foorprint to non-plated ones; - Cut board near SHT4x sensor in order to reduce heat contribution from the rest of the board; - Re-routing; - Added revision number on silkscreen; - Shrunk components ID on silkscreen.
Parts:
- removed TP1: DP, TestPoint:TestPoint_Pad_D1.0mm, symbol Connector:TestPoint
- removed TP2: DN, TestPoint:TestPoint_Pad_D1.0mm, symbol Connector:TestPoint
Connections:
- net at J1.A6 (DP1): no longer J1.B6 (DP2)
- net at J1.A7 (DN1): no longer J1.B7 (DN2)
- no-connect marks 6 -> 10
